File: SmartwatchProject.kicad_sch (KiCad schematic)
At the start: 17 parts, among them SW1 SW_Push, SW2 SW_Push, U1 ESP32-S3-WROOM-1, U2 DS3231M, U3 ADXL345BCCZ, U4 DRV2605LDGSR, U5 XPT2046QF, U6 MAX98357A, U7 2478

Commit message: Net update
Connections:
- net GND: now also U3.11 (RESERVED_GND)
- net VS: now reaches U3.3 (RESERVED_VS)
- net VS: now also U3.6 (VS)
Changed lines of the file:
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@@
+	(wire
+		(pts
+			(xy 132.08 39.37) (xy 137.16 39.37)
+		)
+		(stroke
+			(width 0)
+			(type default)
+		)
+	)
 	(wire
 		(pts
@@
 	(wire
 		(pts
+			(xy 132.08 36.83) (xy 137.16 36.83)
+		)
+		(stroke
+			(width 0)
+			(type default)
+		)
+	)
+	(wire
+		(pts
 			(xy 241.3 153.67) (xy 245.11 153.67)
 		)
@@
 		(pts
 			(xy 187.96 21.59) (xy 190.5 21.59)
+		)
+		(stroke
+			(width 0)
+			(type default)
+		)
+	)
+	(wire
+		(pts
+			(xy 187.96 19.05) (xy 191.77 19.05)
 		)
 		(stroke
@@
 		)
 	)
+	(label "VS"
+		(at 132.08 36.83 0)
+		(effects
+			(font
+				(size 1.27 1.27)
+			)
+			(justify left bottom)
+		)
+	)
 	(label "IO3"
 		(at 177.8 76.2 180)
@@
 	)
 	(label "GND"
+		(at 132.08 39.37 0)
+		(effects
+			(font
+				(size 1.27 1.27)
+			)
+			(justify left bottom)
+		)
+	)
+	(label "GND"
 		(at 191.77 46.99 0)
 		(effects
@@
 		(effects
 			(font
+				(size 1.27 1.27)
+			)
+			(justify right bottom)
+		)
+	)
+	(label "VS"
+		(at 191.77 19.05 180)
+		(effects
+			(font
