File: SmartwatchProject.kicad_sch (KiCad schematic)
At the start: 17 parts, among them SW1 SW_Push, SW2 SW_Push, U1 ESP32-S3-WROOM-1, U2 DS3231M, U3 ADXL345BCCZ, U4 DRV2605LDGSR, U5 XPT2046QF, U6 MAX98357A, U7 2478

Commit message: SecondCommit
Parts:
- added BT1: Battery_Cell, symbol Device:Battery_Cell
- added C3: 10uF, symbol Device:C
- added C4: 22uF, symbol Device:C
- added C5: 1uF, symbol Device:C
- added C6: 0.1uF, symbol Device:C
- added J1: USB_B_Micro, Connector_USB:USB_Micro-B_Molex-105017-0001, symbol Connector:USB_B_Micro
- added R5: 2k, symbol Device:R_US
- added U8: AMS1117-3.3, Package_TO_SOT_SMD:SOT-223-3_TabPin2, symbol Regulator_Linear:AMS1117-3.3
- added U9: MCP73831-2-MC, Package_DFN_QFN:DFN-8-1EP_3x2mm_P0.5mm_EP1.7x1.4mm, symbol Battery_Management:MCP73831-2-MC
Connections:
- net +3.3V: now also C4.2, C5.1, C6.1, U8.2 (VO)
- net GND: now also U3.11 (RESERVED_GND), BT1.2 (-), C3.2, C4.1, C5.2, C6.2, J1.5 (GND), J1.6 (Shield), R5.2, U8.1 (GND)
- net INT: now also U1.23 (IO21); no longer U1.14 (USB_D+)
- net GAIN: now reaches U6.2 (GAIN_SLOT)
- net GAIN: now also U1.5 (IO5)
- net SD MODE: now reaches U6.4 (~{SD_MODE})
- net SD MODE: now also U1.27 (IO0)
- net VS: now reaches U3.3 (RESERVED_VS)
- net VS: now also U3.6 (VS)
- net D-: now reaches U1.13 (USB_D-)
- net D-: now also J1.2 (D-)
- new net: R5.1, U9.8 (PROG)
- new net: U9.1 (V_{DD}), U9.2 (V_{DD})
- new net D+: J1.3 (D+), U1.14 (USB_D+)
- new net USB5V: BT1.1 (+), C3.1, J1.1 (VBUS), U8.3 (VI), U9.3 (V_{BAT}), U9.4 (V_{BAT})
- no-connect marks 0 -> 1
Other:
- note added: "Power & Program"
- moved on the sheet: LS1, U6, U7

Commit message: ThirdCommit
Parts:
- removed U5: XPT2046QF, Package_DFN_QFN:QFN-16-1EP_4x4mm_P0.65mm_EP2.1x2.1mm, symbol Driver_Display:XPT2046QF
- removed U7: 2478, 2478:ADAFRUIT_2478, symbol 2478:2478
- added J2: SM13B-GHS-TB_LF__SN_, SM13B-GHS-TB_LF__SN_:JST_SM13B-GHS-TB_LF__SN_, symbol SM13B-GHS-TB_LF__SN_:SM13B-GHS-TB_LF__SN_
Connections:
- net GND: now also J2.SH1 (SHIELD), J2.SH2 (SHIELD)

Commit message: Some small edits
Parts:
- C1: footprint (none) -> Capacitor_SMD:C_0603_1608Metric
Changed lines of the file:
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@@
 			)
 		)
-		(property "Footprint" ""
+		(property "Footprint" "Capacitor_SMD:C_0603_1608Metric"
 			(at 46.99 15.5448 0)
 			(effects

Commit message: FourthCommit
Parts:
- added C7, C8, C9: 10uF, symbol Device:C
- R3, R4: value 4.7k -> 10k
Connections:
- net RST1 is gone; now on net RST: R3.2, SW1.2, U2.4 (~{RST})
- net +3.3V: now also C7.1, C8.2, C9.1
- net GND: now also C7.2, C8.1, C9.2
- net SD MODE: now also U1.12 (IO8); no longer U1.27 (IO0)
- net RST: now reaches U1.3 (EN)
- net RST2 renamed BOOT
- net BOOT: now also U1.27 (IO0)
Other:
- note added: "BOOT Button"
- note added: "RST Button"
- note removed: "RST Button1"
- note removed: "RST Button2"
- moved on the sheet: J2

Commit message: FifthCommit
Parts:
- added R6, R7: 0, symbol Device:R_US
Connections:
- net IRQ is gone; now on net INT: U1.4 (IO4)
- net +3.3V: now also R6.1
- net GND: now also U6.17 (PAD), R7.1
- net INT: no longer U1.23 (IO21)
- net GAIN: no longer names the net of U6.2 (GAIN_SLOT)
- net GAIN: now also R6.2, R7.2; no longer U1.5 (IO5)
- no-connect marks 1 -> 2

Commit message: SixthCommit
Parts:
- added R8: 1M, symbol Device:R_US
Connections:
- net SD MODE: now also R8.1; no longer U6.4 (~{SD_MODE})
- new net: R8.2, U6.4 (~{SD_MODE})
Other:
- moved on the sheet: C5, C6, LS1, R6, R7, U6

Commit message: Schematic Update
Connections:
- net MISO: now also J2.3
- net MOSI: now also J2.4
Other:
- note added: "Microcontroller"

Commit message: v1
Parts:
- removed U1: ESP32-S3-WROOM-1, RF_Module:ESP32-S3-WROOM-1, symbol RF_Module:ESP32-S3-WROOM-1
- added AE1: Antenna_Chip, symbol Device:Antenna_Chip
- added C10, C11, C20, C21: TBD, symbol Device:C
- added C12, C15, C16: 0.1uF, symbol Device:C
- added C13, C17, C18: 1uF, symbol Device:C
- added C14: 10uF, symbol Device:C
- added C19: 10nF, symbol Device:C
- added L1, L2: 0.2nH, symbol Device:L
- added L3: TBD, symbol Device:L
- added R10, R11, R12, R13, R9: 0, symbol Device:R_US
- added R14: 499, symbol Device:R_US
- added U5: ESP32-C3, Package_DFN_QFN:QFN-32-1EP_5x5mm_P0.5mm_EP3.7x3.7mm, symbol MCU_Espressif:ESP32-C3
- added U7: W25Q32JVSS, Package_SO:SOIC-8_5.3x5.3mm_P1.27mm, symbol Memory_Flash:W25Q32JVSS
- added Y1: 40MHz, symbol Device:Crystal
Connections:
- net CS: now also U5.21 (SPICS0), U7.1 (~{CS})
- net D+: now also U5.6 (GPIO2)
- net D-: now also U5.8 (GPIO3)
- net GND: now also AE1.2 (PCB_Trace), C10.2, C11.2, C12.2, C13.2, C14.2, C15.2, C16.2, C17.2, C18.1, C19.1, C20.2, C21.2, U5.33 (GND), U7.4 (GND); no longer U4.4 (IN/TRIG)
- net MISO: now also R13.2, U7.2 (DO/IO_{1})
- net MOSI: now also R12.2, U7.5 (DI/IO_{0})
- net RST: now also U5.7 (CHIP_EN)
- net SCK: now also R11.2, U7.6 (CLK)
- net SCL: now also U5.15 (GPIO9)
- net SDA: now also U5.14 (GPIO8)
- net IO2 renamed Haptic_EN
- new net: C13.1, L2.1, U5.2 (VDD3P3), U5.3 (VDD3P3)
- new net: C10.1, L1.1, U5.1 (LNA_IN)
- new net: R9.1, U5.19 (SPIHD)
- new net: R10.1, U5.20 (SPIWP)
- new net: R11.1, U5.22 (SPICLK)
- new net: R12.1, U5.23 (SPID)
- new net: R13.1, U5.24 (SPIQ)
- new net: R14.2, U5.28 (U0TXD)
- new net: C20.1, U5.29 (XTAL_N), Y1.2
- new net: L3.2, U5.30 (XTAL_P)
- new net: AE1.1 (FEED), C11.1, L1.2
- new net: C21.1, L3.1, Y1.1
- new net LSPIWP: R10.2, U7.3 (~{WP}/IO_{2})
- new net MTCK: U5.12 (MTCK)
- new net MTDI: U5.10 (MTDI)
- new net MTDO: U5.13 (MTDO)
- new net MTMS: U5.9 (MTMS)
- new net SPIHD: R9.2, U7.7 (~{HOLD}/~{RESET}/IO_{3})
- new net TBD: C12.1, C14.1, C15.1, C16.1, C17.1, C18.2, C19.2, L2.2, U5.11 (VDD3P3_RTC), U5.17 (VDD3P3_CPU), U5.18 (VDD_SPI), U5.31 (VDDA), U5.32 (VDDA), U7.8 (VCC)
- new net U0RXD: U5.27 (U0RXD)
- new net U0TXD: R14.1
- new net XTAL_32K_N: U5.5 (XTAL_32K_N)
- new net XTAL_32K_P: U5.4 (XTAL_32K_P)
- no-connect marks 2 -> 3
Other:
- note added: "Flash"
- note removed: "Microcontroller"
- moved on the sheet: B1, BT1, C1, C2, C3, C4, C5, C6, C7, C8, C9, J1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
