File: SmartwatchProject.kicad_sch (KiCad schematic)
At the start: 58 parts, among them J1 USB_B_Micro, J2 SM13B-GHS-TB_LF__SN_, Q1 AO3401A, SW1 SW_Push, SW2 SW_Push, U1 CH340C, U2 DS3231M, U4 DRV2605LDGSR, U5 ESP32-C3, U6 MAX98357A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

Commit message: small changes
Connections:
- net XTAL_32K_N: no longer names the net of U5.5 (XTAL_32K_N)
- net XTAL_32K_P: no longer names the net of U5.4 (XTAL_32K_P)
- no-connect marks 17 -> 21
Other:
- note removed: "What are these 2 pins used for?"

Commit message: PCB Draft
Parts:
- removed LS1: CMS-16098A-SP, CMS-16098A-SP:CUI_CMS-16098A-SP, symbol CMS-16098A-SP:CMS-16098A-SP
- removed U9: MCP73831-2-MC, Package_DFN_QFN:DFN-8-1EP_3x2mm_P0.5mm_EP1.7x1.4mm, symbol Battery_Management:MCP73831-2-MC
- added LS1: CMS-16098A-SP, Imports_Global:CUI_CMS-16098A-SP, symbol Imports:CMS-16098A-SP
- added U3: MCP73831-2-MC, Package_DFN_QFN:DFN-8-1EP_3x2mm_P0.5mm_EP1.7x1.4mm, symbol Imports:MCP73831-2-MC
- AE1: value Antenna_Chip -> AMCA31-2R450G-S1F-T3; footprint (none) -> Imports_Global:XDCR_AMCA31-2R450G-S1F-T3
- BT1: footprint (none) -> Connector_PinHeader_1.00mm:PinHeader_1x02_P1.00mm_Vertical
- C10, C11, C12, C13, C14, C15, C16, C17, C18, C19, C2, C20, C21, C3, C4, C5, C6, C7, C8: footprint (none) -> Capacitor_SMD:C_0402_1005Metric
- J2: footprint SM13B-GHS-TB_LF__SN_:JST_SM13B-GHS-TB_LF__SN_ -> Imports_Global:JST_SM13B-GHS-TB_LF__SN_
- L1, L2, L3: footprint (none) -> Inductor_SMD:L_0402_1005Metric
- R1, R10, R11, R12, R13, R14, R15, R16, R2, R3, R4, R5, R6, R7, R8, R9: footprint (none) -> Resistor_SMD:R_0402_1005Metric
- SW1, SW2: footprint (none) -> Button_Switch_SMD:SW_SPST_TL3342
- Y1: footprint (none) -> Crystal:Crystal_SMD_3215-2Pin_3.2x1.5mm
Connections:
- net BOOT: no longer U1.13 (~{DTR}), U5.15 (GPIO9)
- net GND: now also AE1.1 (FEED), U3.6 (V_{SS}), U3.9 (Thermal); no longer AE1.2 (PCB_Trace)
- net USB5V: now also U3.1 (V_{DD}), U3.2 (V_{DD})
- net at U6.10 (OUTN): now also LS1.N
- net at U6.9 (OUTP): now also LS1.P
- net at BT1.1 (+), C8.1, Q1.3 (D): now also U3.3 (V_{BAT}), U3.4 (V_{BAT})
- net at C11.1, L1.2: now also AE1.2 (PCB_Trace); no longer AE1.1 (FEED)
- net at R5.1: now also U3.8 (PROG)

Commit message: Schematic Draft
Connections:
- net BCLK: now also U5.6 (GPIO2); no longer U5.8 (GPIO3)
- net CS: no longer J2.6
- net DC: now also U5.26 (GPIO19); no longer U5.16 (GPIO10)
- net DIN: now also U5.16 (GPIO10); no longer U5.6 (GPIO2)
- net LRCLK: now also U5.8 (GPIO3); no longer U5.14 (GPIO8)
- net SCL: now also U5.15 (GPIO9); no longer U5.26 (GPIO19)
- net SDA: now also U5.14 (GPIO8); no longer U5.25 (GPIO18)
- new net Display_CS: J2.6, U5.25 (GPIO18)
Changed lines of the file:
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@@
-		)
-	)
-	(label "LRCLK"
-		(at 58.42 147.32 180)
-		(effects
-			(font
-				(size 1.27 1.27)
-			)
-			(justify right bottom)
 		)
 	)
@@
 		)
 	)
+	(label "DIN"
+		(at 58.42 152.4 180)
+		(effects
+			(font
+				(size 1.27 1.27)
+			)
+			(justify right bottom)
+		)
+	)
 	(label "CS"
 		(at 116.84 170.18 0)
@@
 		)
 	)
-	(label "BCLK"
-		(at 58.42 144.78 180)
-		(effects
-			(font
-				(size 1.27 1.27)
-			)
-			(justify right bottom)
-		)
-	)
 	(label "D-"
 		(at 153.67 31.75 180)
@@
 		)
 	)
-	(label "SDA"
-		(at 58.42 154.94 180)
-		(effects
-			(font
-				(size 1.27 1.27)
-			)
-			(justify right bottom)
-		)
-	)
 	(label "USB5V"
 		(at 167.64 16.51 0)
@@
 		)
 	)
-	(label "SCL"
+	(label "DC"
 		(at 58.42 157.48 180)
 		(effects
@@
 		)
 	)
+	(label "SDA"
+		(at 58.42 147.32 180)
+		(effects
+			(font
+				(size 1.27 1.27)
+			)
+			(justify right bottom)
+		)
+	)
 	(label "D-"
 		(at 123.19 78.74 180)
@@
 		)
 	)
+	(label "BCLK"
+		(at 58.42 142.24 180)
+		(effects
+			(font
+				(size 1.27 1.27)
+			)
+			(justify right bottom)
+		)
+	)
+	(label "Display_CS"
+		(at 58.42 154.94 180)
+		(effects
+			(font
+				(size 1.27 1.27)
+			)
+			(justify right bottom)
+		)
+	)
 	(label "SPIHD"
 		(at 116.84 165.1 0)
@@
 		)
 	)
-	(label "DIN"
-		(at 58.42 142.24 180)
-		(effects
-			(font
-				(size 1.27 1.27)
-			)
-			(justify right bottom)
-		)
-	)
-	(label "DC"
-		(at 58.42 152.4 180)
-		(effects
-			(font
-				(size 1.27 1.27)
-			)
-			(justify right bottom)
-		)
-	)
 	(label "RST"
 		(at 143.51 88.9 0)
@@
 		)
 	)
+	(label "LRCLK"
+		(at 58.42 144.78 180)
+		(effects
+			(font
+				(size 1.27 1.27)
+			)
+			(justify right bottom)
+		)
+	)
 	(label "TXD"
 		(at 143.51 68.58 0)
@@
 		)
 	)
+	(label "SCL"
+		(at 58.42 149.86 180)
+		(effects
+			(font
+				(size 1.27 1.27)
+			)
+			(justify right bottom)
+		)
+	)
 	(label "SDA"
 		(at 156.21 74.93 180)
@@
 		)
 	)
-	(label "CS"
+	(label "Display_CS"
 		(at 255.27 44.45 90)
 		(effects
